Commit message: Task 2: Completed

File: my_rb1_description/urdf/my_rb1_robot.xacro (robot description, xacro)
@@ -1,4 +1,6 @@
 <?xml version="1.0"?>
 <robot name="rb1" xmlns:xacro="http://www.ros.org/wiki/xacro">
+    <xacro:include filename="$(find my_rb1_description)/urdf/my_rb1_robot.gazebo" />
+    <!-- Materials -->
     <material name="blue">
         <color rgba="0 0 1 1"/>
@@ -10,4 +12,5 @@
         <color rgba="0.5 0.5 0.5 1"/>
     </material>
+    <!-- Macros for Inertia -->
     <xacro:macro name="cylinder_inertia" params="m r h xyz rpy">
         <inertial>
@@ -28,6 +31,6 @@
         </inertial>
     </xacro:macro>
+    <!-- Base Link -->
     <link name="base_footprint" />
-    <!-- Base Link -->
     <link name="base_link">
         <visual>
@@ -38,6 +41,12 @@
             <material name="blue" />
         </visual>
+        <collision>
+            <geometry>
+                <cylinder radius="0.25" length="0.3" />
+            </geometry>
+            <origin xyz="0 0 0" rpy="0 0 0" />
+        </collision>
         <xacro:cylinder_inertia m="19.5" r="0.25" h="0.3"
-                                            xyz="0 0 0" rpy="0 0 0" />
+                                xyz="0 0 0" rpy="0 0 0" />
     </link>
     <joint name="base_joint" type="fixed">
@@ -55,6 +64,12 @@
             <material name="red" />
         </visual>
+        <collision>
+            <geometry>
+                <cylinder radius="0.025" length="0.05"/>
+            </geometry>
+            <origin xyz="0 0 0" rpy="0 0 0" />
+        </collision>
         <xacro:cylinder_inertia m="1.25" r="0.025" h="0.05"
-                                            xyz="0 0 0" rpy="0 0 0" />
+                                xyz="0 0 0" rpy="0 0 0" />
     </link>
     <joint name="left_wheel_joint" type="continuous">
@@ -72,6 +87,12 @@
             <material name="red" />
         </visual>
+        <collision>
+            <geometry>
+                <cylinder radius="0.025" length="0.05"/>
+            </geometry>
+            <origin xyz="0 0 0" rpy="0 0 0" />
+        </collision>
         <xacro:cylinder_inertia m="1.25" r="0.025" h="0.05"
-                                            xyz="0 0 0" rpy="0 0 0" />
+                                xyz="0 0 0" rpy="0 0 0" />
     </link>
     <joint name="right_wheel_joint" type="continuous">
@@ -89,4 +110,10 @@
             <material name="gray" />
         </visual>
+        <collision>
+            <geometry>
+                <sphere radius="0.025"/>
+            </geometry>
+            <origin xyz="0 0 0" rpy="0 0 0" />
+        </collision>
         <xacro:sphere_inertia m="1.25" r="0.025" xyz="0 0 0" rpy="0 0 0" />
     </link>
@@ -103,4 +130,10 @@
             <material name="gray" />
         </visual>
+        <collision>
+            <geometry>
+                <sphere radius="0.025"/>
+            </geometry>
+            <origin xyz="0 0 0" rpy="0 0 0" />
+        </collision>
         <xacro:sphere_inertia m="1.25" r="0.025" xyz="0 0 0" rpy="0 0 0" />
     </link>
@@ -119,6 +152,12 @@
             <material name="red" />
         </visual>
+        <collision>
+            <geometry>
+                <cylinder radius="0.02" length="0.03"/>
+            </geometry>
+            <origin xyz="0 0 0" rpy="0 0 0" />
+        </collision>
         <xacro:cylinder_inertia m="0.5" r="0.02" h="0.03"
-                                            xyz="0 0 0" rpy="0 0 0" />
+                                xyz="0 0 0" rpy="0 0 0" />
     </link>
     <joint name="front_laser_joint" type="fixed">
